Commit message: Aggiunti nuovi pkg
Ogni modulo si trova in un pkg separato

File: src/my_robot/robot_description/robot_description.xacro (robot description, xacro)
@@ -34,9 +34,15 @@
     <xacro:property name="imu_frame_orientation"            value="0 0 0"/>
     <!-- Import Rviz colors -->
-    <xacro:include filename="$(find robot_pkg)/models/materials.xacro"/>
+    <xacro:include filename="$(find my_robot)/robot_description/materials.xacro"/>
     <!-- Import Gazebo customization elemets -->
-    <xacro:include filename="$(find robot_pkg)/models/robot_description.gazebo"/>
+    <xacro:include filename="$(find my_robot)/robot_description/robot_description.gazebo"/>
     <!-- Import laser sensor -->
-    <xacro:include filename="$(find robot_pkg)/models/sensors/hokuyo.urdf.xacro"/>
+    <xacro:include filename="$(find my_robot)/sensors/hokuyo.urdf.xacro"/>
+    <!-- Extra link (non-inertial) -->
+    <link name="base_footprint" />
+    <joint name="base_footprint_joint" type="fixed">
+        <parent link="base_footprint" />
+        <child link="base_link" />
+    </joint>
     <!-- Chassis Link -->
     <link name="base_link">

Commit message: Riordinato file urdf

File: src/my_robot/robot_description/robot_description.xacro (robot description, xacro)
@@ -29,5 +29,5 @@
     <xacro:property name="rear_wheel_frame_position"        value="${-body_lenght/2 + 2 * rear_wheel_radius} 0 ${-rear_wheel_radius}"/>
     <xacro:property name="rear_wheel_frame_orientation"     value="0 0 0"/>
-    <xacro:property name="laser_frame_position"             value="0 0 ${body_height}"/>
+    <xacro:property name="laser_frame_position"             value="0 0 ${body_height + 0.02}"/>
     <xacro:property name="laser_frame_orientation"          value="0 0 0"/>
     <xacro:property name="imu_frame_position"               value="0 0 ${body_height/2}"/>
@@ -39,4 +39,6 @@
     <!-- Import laser sensor -->
     <xacro:include filename="$(find my_robot)/sensors/hokuyo.urdf.xacro"/>
+    <!-- Import IMU sensor -->
+    <xacro:include filename="$(find my_robot)/sensors/imu.urdf.xacro"/>
     <!-- Extra link (non-inertial) -->
     <link name="base_footprint" />
@@ -69,17 +71,14 @@
         </inertial>
     </link>
-    <!-- IMU Link -->
-    <link name="imu_link">
-        <inertial>
-        <mass value="0.001"/>
-        <origin xyz="0 0 0" rpy="0 0 0"/>
-        <inertia ixx="${dummy_inertia}" ixy="0.0" ixz="0.0" iyy="${dummy_inertia}" iyz="0.0" izz="${dummy_inertia}"/>
-        </inertial>
-    </link>
-    <joint name="imu_joint" type="fixed">
-        <parent link="base_link" />
-        <child link="imu_link" />
-        <origin xyz="${imu_frame_position}" rpy="${imu_frame_orientation}"/>
-    </joint>
+     <!-- IMU link -->
+    <xacro:imu xyz="${imu_frame_position}"
+        rpy="${imu_frame_orientation}"
+        parent="base_link">
+    </xacro:imu>
+    <!-- Laser link -->
+    <xacro:hokuyo_laser xyz="${laser_frame_position}"
+        rpy="${laser_frame_orientation}"
+        parent="base_link">
+    </xacro:hokuyo_laser>
     <!-- Right wheel joint -->
     <joint name="right_wheel_joint" type="continuous">
@@ -206,9 +205,4 @@
         </inertial>
     </link>
-    <!-- Laser link -->
-    <xacro:hokuyo_laser xyz="0 0 ${body_height + 0.02}"
-        rpy=" 0 0 0"
-        parent="base_link">
-    </xacro:hokuyo_laser>
     <!-- Transmission at joints-->
     <transmission name="right_wheel_trans">
@@ -232,29 +226,3 @@
         </actuator>
     </transmission>
-    <!-- Gazebo differential drive plugin -->
-    <gazebo>
-        <plugin name="differential_drive_controller" filename="libgazebo_ros_diff_drive.so">
-            <robotNamespace>/$(arg namespace)</robotNamespace>
-            <alwaysOn>true</alwaysOn>
-            <legacyMode>false</legacyMode>
-            <updateRate>50</updateRate>
-            <leftJoint>left_wheel_joint</leftJoint>
-            <rightJoint>right_wheel_joint</rightJoint>
-            <wheelSeparation>${body_width + control_wheel_lenght}</wheelSeparation>
-            <wheelDiameter>${2 * control_wheel_radius}</wheelDiameter>
-            <wheelTorque>10</wheelTorque>
-            <commandTopic>cmd_vel</commandTopic>
-            <odometryTopic>odom</odometryTopic>
-            <odometryFrame>$(arg namespace)/odom</odometryFrame>
-            <robotBaseFrame>$(arg namespace)/base_link</robotBaseFrame>
-            <publishWheelTF>false</publishWheelTF>
-            <publishOdomTF>true</publishOdomTF>
-            <publishWheelJointState>true</publishWheelJointState>
-            <wheelAcceleration>0</wheelAcceleration>
-            <odometrySource>world</odometrySource>
-            <wheelAcceleration>1</wheelAcceleration>
-            <publishTf>1</publishTf>
-            <rosDebugLevel>na</rosDebugLevel>
-        </plugin>
-    </gazebo>
 </robot>

File: src/my_robot/sensors/hokuyo.urdf.xacro (robot description, xacro)
@@ -28,37 +28,4 @@
         </inertial>
     </link>
-    <gazebo reference="hokuyo_laser_link">
-        <gravity>true</gravity>
-        <sensor type="ray" name="head_hokuyo_sensor">
-            <pose>0 0 0 0 0 0</pose>
-            <visualize>false</visualize>
-            <update_rate>40</update_rate>
-            <ray>
-                <scan>
-                    <horizontal>
-                        <samples>360</samples>
-                        <resolution>1</resolution>
-                        <min_angle>-3.14159</min_angle>
-                        <max_angle>3.14159</max_angle>
-                    </horizontal>
-                </scan>
-                <range>
-                    <min>0.2</min>
-                    <max>20</max>
-                    <resolution>0.025</resolution>
-                </range>
-                <noise>
-                    <type>gaussian</type>
-                    <mean>0.0</mean>
-                    <stddev>0.0</stddev>
-                </noise>
-            </ray>
-            <plugin name="gazebo_ros_head_hokuyo_controller" filename="libgazebo_ros_laser.so">
-                <robotNamespace> /$(arg namespace) </robotNamespace>
-                <topicName>laser_scan</topicName>
-                <frameName>$(arg namespace)/hokuyo_laser_link</frameName>
-            </plugin>
-        </sensor>
-    </gazebo>
 </xacro:macro>
 </robot>

Commit message: aggiunto world

File: src/my_robot/robot_description/robot_description.xacro (robot description, xacro)
@@ -42,9 +42,9 @@
     <xacro:include filename="$(find my_robot)/sensors/imu.urdf.xacro"/>
     <!-- Extra link (non-inertial) -->
-    <link name="base_footprint" />
+    <!-- <link name="base_footprint" />
     <joint name="base_footprint_joint" type="fixed">
         <parent link="base_footprint" />
         <child link="base_link" />
-    </joint>
+    </joint> -->
     <!-- Chassis Link -->
     <link name="base_link">

Commit message: Quasi sistemato move_base

File: src/my_robot/robot_description/robot_description.xacro (robot description, xacro)
@@ -6,18 +6,18 @@
     <xacro:property name="dummy_inertia"                value="1e-09"/>
     <!-- Classic parameters -->
-    <xacro:property name="body_mass"    value="10"/>
-    <xacro:property name="body_lenght"  value="0.7"/>
-    <xacro:property name="body_width"   value="0.4"/>
-    <xacro:property name="body_height"  value="0.3"/>
+    <xacro:property name="body_mass"    value="5"/>
+    <xacro:property name="body_lenght"  value="0.35"/>
+    <xacro:property name="body_width"   value="0.2"/>
+    <xacro:property name="body_height"  value="0.1"/>
+    <!-- Control wheels parameters -->
+    <xacro:property name="control_wheel_mass"   value="2"/>
+    <xacro:property name="control_wheel_radius" value="0.05"/>
+    <xacro:property name="control_wheel_lenght" value="0.03"/>
     <!-- Front wheel parameters -->
     <xacro:property name="front_wheel_mass"     value="0.001"/>
-    <xacro:property name="front_wheel_radius"   value="0.05"/>
+    <xacro:property name="front_wheel_radius"   value="0.025"/>
     <!-- Rear wheel parameters -->
     <xacro:property name="rear_wheel_mass"      value="0.001"/>
-    <xacro:property name="rear_wheel_radius"    value="0.05"/>
-    <!-- Control wheels parameters -->
-    <xacro:property name="control_wheel_mass"   value="2"/>
-    <xacro:property name="control_wheel_radius" value="0.1"/>
-    <xacro:property name="control_wheel_lenght" value="0.1"/>
+    <xacro:property name="rear_wheel_radius"    value="0.025"/>
     <!-- Frame position and orientation -->
     <xacro:property name="right_wheel_frame_position"       value="0 ${-body_width/2 - control_wheel_lenght/2} 0"/>

Commit message: Fine giornata di bestemmie

File: src/my_robot/robot_description/robot_description.xacro (robot description, xacro)
@@ -6,18 +6,18 @@
     <xacro:property name="dummy_inertia"                value="1e-09"/>
     <!-- Classic parameters -->
-    <xacro:property name="body_mass"    value="5"/>
-    <xacro:property name="body_lenght"  value="0.35"/>
-    <xacro:property name="body_width"   value="0.2"/>
-    <xacro:property name="body_height"  value="0.1"/>
+    <xacro:property name="body_mass"    value="2"/>
+    <xacro:property name="body_lenght"  value="0.15"/>
+    <xacro:property name="body_width"   value="0.1"/>
+    <xacro:property name="body_height"  value="0.05"/>
     <!-- Control wheels parameters -->
-    <xacro:property name="control_wheel_mass"   value="2"/>
-    <xacro:property name="control_wheel_radius" value="0.05"/>
-    <xacro:property name="control_wheel_lenght" value="0.03"/>
+    <xacro:property name="control_wheel_mass"   value="0.5"/>
+    <xacro:property name="control_wheel_radius" value="0.04"/>
+    <xacro:property name="control_wheel_lenght" value="0.02"/>
     <!-- Front wheel parameters -->
     <xacro:property name="front_wheel_mass"     value="0.001"/>
-    <xacro:property name="front_wheel_radius"   value="0.025"/>
+    <xacro:property name="front_wheel_radius"   value="0.02"/>
     <!-- Rear wheel parameters -->
     <xacro:property name="rear_wheel_mass"      value="0.001"/>
-    <xacro:property name="rear_wheel_radius"    value="0.025"/>
+    <xacro:property name="rear_wheel_radius"    value="0.02"/>
     <!-- Frame position and orientation -->
     <xacro:property name="right_wheel_frame_position"       value="0 ${-body_width/2 - control_wheel_lenght/2} 0"/>
